File: KiCAD_files/InverterLeg.kicad_sch (KiCad schematic)
At the start: 72 parts, among them J801 Conn_Coaxial_Small, J802 Conn_Coaxial_Small, J803 Conn_01x01_Pin, J804 Conn_01x03_Socket, J806 Conn_01x01_Pin, J811 Screw_Terminal_01x01, J814 Screw_Terminal_01x01, J817 Screw_Terminal_01x01, J825 HC-PBB08-2-08-M-H4.0-G1-R-P-04, J827 HC-PBB08-2-08-M-H4.0-G1-R-P-04, J831 HC-PBB08-2-08-M-H4.0-G1-R-P-04, Q801 IPT60R055CM8, Q802 IPT60R055CM8, T801 CMB1670V, T802 CMB1670V, U704 VPS8701B, U707 VPS8701B, U801 LT1761-SD, U802 LT1761-SD, U811 TMP117xxDRV, U815 TMP117xxDRV

Commit message: schematic tidy-up and traces wip
Parts:
- added TP801, TP802, TP803, TP804, TP805, TP806, TP807, TP808, TP809, TP810, TP811, TP812, TP813, TP814, TP815, TP816, TP817, TP818, TP819, TP820, TP821, TP822: (no value), TestPoint:TestPoint_Pad_D1.0mm, symbol Connector:TestPoint
- U603: value (none) -> ucc21222
Connections:
- net +12V_PGND: now also TP807.1
- net +5V_PGND: now also TP820.1
- net 12V_{HS}: now also TP810.1
- net 12V_{LSRAW}: now also TP814.1
- net 12V_{LS}: now also TP812.1
- net ADDR_HS: now also TP822.1
- net ADDR_LS: now also TP821.1
- net ALERT_HS: now also TP818.1
- net ALERT_LS: now also TP817.1
- net DGND: now also TP804.1
- net DIS: now also TP803.1
- net EN: now also TP805.1
- net K_{GNDLS}: now also TP813.1
- net K_{SWN}: now also TP811.1
- net PGND: now also TP819.1
- net PGND2: now also TP806.1, TP808.1
- net PWMH_{MCU}: now also TP801.1
- net PWML_{MCU}: now also TP802.1
- net SCL_{PWR}: now also TP816.1
- net SDA_{PWR}: now also TP815.1
- net SPEED: now also TP809.1
- net 12V_{HSRAW}: now reaches C734.1, D709.1 (K), D710.1 (K), U801.1 (VIN), U801.3 (~{SHDN})
Other:
- note added: "12V High Side"
- note added: "12V High Side RAW"
- note added: "12V Low Side"
- note added: "12V Low Side RAW"
- note added: "12VP"
- note added: "5VD"
- note added: "5VP"
- note added: "Driver Digital side"
- note added: "Driver High side"
- note added: "Driver Low side"
- note added: "FAN"
- note added: "Isolation"
- note added: "J825"
- note added: "J827"
- note added: "J831"
- note added: "Temp sensors"
- moved on the sheet: C602, C604, C605, C607, C608, C612, C614, C616, C624, C626, C703, C709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

Commit message: nearly no problems left with the pcb. still need a little more work
Parts:
- TP801, TP802, TP803, TP804, TP805, TP806, TP807, TP808, TP809, TP810, TP811, TP812, TP813, TP814, TP815, TP816, TP817, TP818, TP819, TP820, TP821, TP822: footprint TestPoint:TestPoint_Pad_D1.0mm -> Footprints:TestPoint_Pad_D1.0mm_small_courtyard
- U603: value ucc21222 -> (none)
Other:
- note added: "TODO: ref UCC pas la bonne (peut etre UCC21520ADWR)SOIC-16-300mil"

Commit message: HB board is nearly finished for silicium. need to find the driver and maybe change the MOS. the LCSC number are not done and will be processes after the Driver and mos freeze
Parts:
- J825, J827, J831: LCSC C41421136 -> C41421120
- T801, T802: value CMB1670V -> TE1212-2W6ENT
Other:
- note added: "1:1.06"
- note added: "DC"
- note added: "LDO"
- note added: "TODO: ref UCC pas la bonne (peut etre UCC21520ADWR)SOIC-16-300mil FINIR LCSC NUMBER"
- note removed: "TODO: ref UCC pas la bonne (peut etre UCC21520ADWR)SOIC-16-300mil"
- note removed: "WHY only this transformer has an ENABLE signal??"
