File: KiCAD_files/InverterLeg.kicad_sch (KiCad schematic)
At the start: 96 parts, among them J801 AIPEX-4, J802 AIPEX-4, J803 2LC000-739, J804 Conn_01x03_Socket, J806 2LC000-739, J811 SMTSO3050CTJ, J814 SMTSO3050CTJ, J817 SMTSO3050CTJ, J825 HC-PBB08-2-08-M-H1.0-G1-R-P-04, J827 HC-PBB08-2-08-M-H1.0-G1-R-P-04, J831 HC-PBB08-2-08-M-H1.0-G1-R-P-04, Q801 AGM15T05LL, Q802 AGM15T05LL, T801 TE1212-1W6ENT, T802 TE1212-1W6ENT, U603 UCC21520DWR, U704 VPS8701B, U707 VPS8701B, U801 SY6345AAC, U802 SY6345AAC, U803 24C02S(XBLW), U811 T117B, U815 T117B

Commit message: adjusted the values of the 2 12v rails to convert them into 10v rails. This is for not overloading the VGS of the MOS
Parts:
- R610, R612: value 510k -> 158k; LCSC C11616 -> C99856
- R611, R613: value 27k -> 10k; LCSC C25771 -> C2906861
Other:
- note added: "V_{OUT} = 0.6 x (1 + (R610/R611)) V_{OUT} = @{round(0.6 * (1 + (${/8d0c1d66-35ef-4a53-a28f-436a11b54f42/863dab66-1bd6-49ee-8756-763493bfe5e2:Value}/${/8d0c1d66-35ef-4a53-a28f-436a11b54f42/e29cd323-d1f9-4fc6-be36-935751522f90:Value})),2)}V"
- note added: "V_{OUT} = 0.6 x (1 + (R612/R613)) V_{OUT} = @{round(0.6 * (1 + (${/8d0c1d66-35ef-4a53-a28f-436a11b54f42/153ae966-be28-4ef2-b43e-ea2e9beaff1f:Value}/${/8d0c1d66-35ef-4a53-a28f-436a11b54f42/9b8227a6-f6d8-4461-b56f-2b44b0c1a3de:Value})),2)}V"
- note removed: "V_{OUT} = 0.6 x (1 + (R610/R611)) V_{OUT} = @{round(0.6*(1+510000/27000),2)}V"
- note removed: "V_{OUT} = 0.6 x (1 + (R612/R613)) V_{OUT} = @{round(0.6*(1+510000/27000),2)}V"
Changed lines of the file:
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@@
 		)
 	)
-	(text "V_{OUT} = 0.6 x (1 + (R610/R611))\nV_{OUT} = @{round(0.6*(1+510000/27000),2)}V\n"
+	(text "V_{OUT} = 0.6 x (1 + (R610/R611))\nV_{OUT} = @{round(0.6 * (1 + (${/8d0c1d66-35ef-4a53-a28f-436a11b54f42/863dab66-1bd6-49ee-8756-763493bfe5e2:Value}/${/8d0c1d66-35ef-4a53-a28f-436a11b54f42/e29cd323-d1f9-4fc6-be36-935751522f90:Value})),2)}V\n"
 		(exclude_from_sim no)
-		(at 378.714 61.214 0)
+		(at 382.27 60.198 0)
 		(effects
 			(font
@@
 		)
 	)
-	(text "V_{OUT} = 0.6 x (1 + (R612/R613))\nV_{OUT} = @{round(0.6*(1+510000/27000),2)}V\n"
-		(exclude_from_sim no)
-		(at 202.692 62.992 0)
-		(effects
-			(font
-				(size 1.27 1.27)
-			)
-			(justify left)
-		)
-	)
 	(text "The VPS8701B is enabled when EN is floating or pulled up.\nIt is DISABLED when connected to GND"
 		(exclude_from_sim no)
@@
 		)
 	)
+	(text "V_{OUT} = 0.6 x (1 + (R612/R613))\nV_{OUT} = @{round(0.6 * (1 + (${/8d0c1d66-35ef-4a53-a28f-436a11b54f42/153ae966-be28-4ef2-b43e-ea2e9beaff1f:Value}/${/8d0c1d66-35ef-4a53-a28f-436a11b54f42/9b8227a6-f6d8-4461-b56f-2b44b0c1a3de:Value})),2)}V\n"
+		(exclude_from_sim no)
+		(at 217.424 62.738 0)
+		(effects
+			(font
+				(size 1.27 1.27)
+			)
+			(justify left)
+		)
+	)
 	(junction
 		(at 194.31 132.08)
@@
 			)
 		)
-		(property "Value" "510k"
+		(property "Value" "158k"
 			(at 227.838 40.64 0)
 			(show_name no)
@@
 			)
 		)
-		(property "Description" "510 kohm +/-1%, 62.5 mW thick-film resistor, 0402; UNI-ROYAL 0402WGF1783TCE"
+		(property "Description" ""
 			(at 226.06 39.37 0)
 			(hide yes)
@@
 			)
 		)
-		(property "LCSC" "C11616"
+		(property "LCSC" "C99856"
 			(at 226.06 39.37 0)
 			(hide yes)
@@
 			)
 		)
-		(property "Value" "510k"
+		(property "Value" "158k"
 			(at 390.398 38.1 0)
 			(show_name no)
@@
 			)
 		)
-		(property "Description" "510 kohm +/-1%, 62.5 mW thick-film resistor, 0402; UNI-ROYAL 0402WGF1783TCE"
+		(property "Description" ""
 			(at 388.62 36.83 0)
 			(hide yes)
@@
 			)
 		)
-		(property "LCSC" "C11616"
+		(property "LCSC" "C99856"
 			(at 388.62 36.83 0)
 			(hide yes)
@@
 			)
 		)
-		(property "Value" "27k"
+		(property "Value" "10k"
 			(at 227.838 50.8 0)
 			(show_name no)
@@
 			)
 		)
-		(property "Description" "27 kohm +/-1%, 62.5 mW thick-film resistor, 0402; UNI-ROYAL 0402WGF2002TCE"
+		(property "Description" ""
 			(at 226.06 49.53 0)
 			(hide yes)
@@
 			)
 		)
-		(property "LCSC" "C25771"
+		(property "LCSC" "C2906861"
 			(at 226.06 49.53 0)
 			(hide yes)
@@
 			)
 		)
-		(property "Value" "27k"
+		(property "Value" "10k"
 			(at 390.398 50.8 0)
 			(show_name no)
@@
 			)
 		)
-		(property "Description" "27 kohm +/-1%, 62.5 mW thick-film resistor, 0402; UNI-ROYAL 0402WGF2002TCE"
+		(property "Description" ""
 			(at 388.62 49.53 0)
 			(hide yes)
@@
 			)
 		)
-		(property "LCSC" "C25771"
+		(property "LCSC" "C2906861"
 			(at 388.62 49.53 0)
 			(hide yes)
