File: KiCAD_files/InverterLeg.kicad_pcb (KiCad board)
At the start: 4 copper layers, 29 x 73 mm, 100 parts, among them J801 Conn_Coaxial_Small, J802 Conn_Coaxial_Small, J803 Conn_01x01_Pin, J804 Conn_01x03_Socket, J806 Conn_01x01_Pin, J811 Screw_Terminal_01x01, J814 Screw_Terminal_01x01, J817 Screw_Terminal_01x01, J825 HC-PBB08-2-08-M-H4.0-G1-R-P-04, J827 HC-PBB08-2-08-M-H4.0-G1-R-P-04, J831 HC-PBB08-2-08-M-H4.0-G1-R-P-04, Q801 IPT60R055CM8, Q802 IPT60R055CM8, T801 TE1212-2W6ENT, T802 TE1212-2W6ENT, U704 VPS8701B, U707 VPS8701B, U801 LT1761-SD, U802 LT1761-SD, U811 TMP117xxDRV, U815 TMP117xxDRV

Commit message: Added missing LCSC numbers & rotPos. Fixed DRC rules. Moved logo out of galva iso. Revert GND plane modif.
Signed-off-by: Jean Alinei <jean.alinei@owntech.org>
Parts:
- C616: footprint Capacitor_SMD:C_1206_3216Metric -> Capacitor_SMD:C_0805_2012Metric
- C624, C626: value 4.7uF -> 3.3uF
- D601: value PMEG3010CEJ,115 -> PMEG4010
- D602: value ~ -> PMEG4010
- D703, D704, D709, D710: value PMEG3010 -> PMEG4010
- J803, J806: value Conn_01x01_Pin -> ~
- Q801, Q802: value IPT60R055CM8 -> ~
- R601, R603: value 0R -> 1R
- R602, R604: value 2.2R -> 1R
- R607, R608: value 1k -> 10k
- R609: footprint Resistor_SMD:R_0603_1608Metric -> Resistor_SMD:R_0402_1005Metric
- R610, R612: value 176.8k -> 178k
- TJ801, TJ804: value Thermal_Jumper -> ~
- U603: value ~ -> UCC21520
- moved G*** 16.6 mm to (150.4, 99.8)
- moved G*** 15.6 mm to (156.5, 99.8), turned to 0 degrees
- moved C616 0.49 mm to (142.3, 89.4)
Routing:
- net /12V_{LS}: track 12.8 -> 11.4 mm
- removed copper zone on B.Cu, net /K_{SWN}
- removed copper zone on In2.Cu, net /K_{SWN}
